File: L3MON hackpad/L3MON hackpad.kicad_sch (KiCad schematic)
At the start: 0 parts

Commit message: added the wires from the switch to the XIAO RP2040 and added a rotary encoder
Parts:
- added SW1, SW2, SW3, SW4, SW5, SW6: SW_Push, symbol Switch:SW_Push
- added SW8: RotaryEncoder_Switch, symbol Device:RotaryEncoder_Switch
- added U1: XIAO-RP2040-DIP, Module:MOUDLE14P-XIAO-DIP-SMD, symbol Seeed_Studio_XIAO_Series:XIAO-RP2040-DIP
Connections:
- new net: SW4.2, U1.9 (GPIO2/SCK)
- new net: SW6.2, U1.11 (GPIO3/MOSI)
- new net: SW5.2, U1.10 (GPIO4/MISO)
- new net: SW2.2, U1.7 (GPIO0/TX)
- new net: SW1.2, U1.6 (GPIO7/SCL)
- new net: SW3.2, U1.8 (GPIO1/RX)
- new net +5V: U1.14 (VBUS)
- new net GND: SW1.1, SW2.1, SW3.1, SW4.1, SW5.1, SW6.1, U1.13 (GND)
