File: L3MON hackpad/L3MON hackpad.kicad_sch (KiCad schematic)
At the start: 8 parts, among them SW1 SW_Push, SW2 SW_Push, SW3 SW_Push, SW4 SW_Push, SW5 SW_Push, SW6 SW_Push, SW8 RotaryEncoder_Switch, U1 XIAO-RP2040-DIP

Commit message: added more things
Connections:
- net GND: now also SW8.C
- net at SW8.A: now also U1.5 (GPIO6/SDA)
- net at SW8.B: now also U1.4 (GPIO29/ADC3/A3)
Other:
- moved on the sheet: SW1, SW2, SW3, SW4, SW5, SW6, SW8, U1
