File: L3MON hackpad/L3MON hackpad.kicad_sch (KiCad schematic)
At the start: 8 parts, among them SW1 SW_Push, SW2 SW_Push, SW3 SW_Push, SW4 SW_Push, SW5 SW_Push, SW6 SW_Push, SW8 RotaryEncoder_Switch, U1 XIAO-RP2040-DIP

Commit message: made the pcb
Parts:
- added J1: Conn_01x04_Pin, opl2:SSD1306-0.91-OLED-4pin-128x32, symbol Connector:Conn_01x04_Pin
- SW1, SW2, SW3, SW4, SW5, SW6: footprint (none) -> Button_Switch_Keyboard:SW_Cherry_MX_1.00u_PCB
- SW8: footprint (none) -> Rotary_Encoder:RotaryEncoder_Alps_EC11E-Switch_Vertical_H20mm
- U1: footprint Module:MOUDLE14P-XIAO-DIP-SMD -> Seeed Studio XIAO Series Library:XIAO-RP2040-DIP
Connections:
- net +5V: now also J1.2 (Pin_2)
- net GND: now also J1.1 (Pin_1)
- net at U1.5 (GPIO6/SDA): now also J1.4 (Pin_4); no longer SW8.A
- net at SW8.B: now also U1.1 (GPIO26/ADC0/A0); no longer U1.4 (GPIO29/ADC3/A3)
- net at U1.6 (GPIO7/SCL): now also J1.3 (Pin_3); no longer SW1.2
- net at U1.2 (GPIO27/ADC1/A1): now also SW8.A
- net at U1.3 (GPIO28/ADC2/A2): now also SW1.2
Other:
- moved on the sheet: SW1, SW2
