File: L3MON hackpad/_autosave-L3MON hackpad.kicad_pcb (KiCad board)
At the start: 2 copper layers, 80.5 x 54.1 mm, 9 parts, among them J1 Conn_01x04_Pin, SW1 SW_Push, SW2 SW_Push, SW3 SW_Push, SW4 SW_Push, SW5 SW_Push, SW6 SW_Push, SW8 RotaryEncoder_Switch, U1 XIAO-RP2040-DIP

Commit message: made the pcb
Changed lines of the file:
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@@
 	)
 	(segment
-		(start 103.34625 54.61)
-		(end 117.63375 40.3225)
+		(start 126.70375 41.73)
+		(end 128.11125 40.3225)
 		(width 0.2)
 		(layer "F.Cu")
@@
 	)
 	(segment
-		(start 117.63375 40.3225)
-		(end 128.11125 40.3225)
+		(start 103.34625 54.61)
+		(end 103.4 54.61)
 		(width 0.2)
 		(layer "F.Cu")
+		(net 5)
+	)
+	(segment
+		(start 103.4 54.61)
+		(end 116.28 41.73)
+		(width 0.2)
+		(layer "F.Cu")
+		(net 5)
+	)
+	(segment
+		(start 116.28 41.73)
+		(end 126.70375 41.73)
+		(width 0.2)
+		(layer "F.Cu")
