File: L3MON hackpad/L3MON hackpad.kicad_pcb (KiCad board)
At the start: 2 copper layers, 80.5 x 54.1 mm, 9 parts, among them J1 Conn_01x04_Pin, SW1 SW_Push, SW2 SW_Push, SW3 SW_Push, SW4 SW_Push, SW5 SW_Push, SW6 SW_Push, SW8 RotaryEncoder_Switch, U1 XIAO-RP2040-DIP

Commit message: finished pcb
Parts:
- added G***: LOGO, opl2:front, F.Cu at (104.9, 38.7)
Other:
- board text added: "Hackpad L3M0N"
- board text added: "Place XIAO here"
