File: L3MON hackpad/PCB/L3MON hackpad.kicad_pcb (KiCad board)
At the start: 2 copper layers, 80.5 x 54.1 mm, 10 parts, among them J1 Conn_01x04_Pin, SW1 SW_Push, SW2 SW_Push, SW3 SW_Push, SW4 SW_Push, SW5 SW_Push, SW6 SW_Push, SW8 RotaryEncoder_Switch, U1 XIAO-RP2040-DIP

Commit message: finished the code
Routing:
- net GND: track 150.0 -> 154.0 mm
- net Net-(J1-Pin_4): track 38.6 -> 35.8 mm, vias 0 -> 1
- net Net-(U1-GPIO2/SCK): track 27.1 -> 28.2 mm, vias 0 -> 1
Changed lines of the file:
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@@
-	)
-	(segment
-		(start 169.2275 52.07)
-		(end 164.93025 47.77275)
-		(width 0.2)
-		(layer "F.Cu")
-		(net 2)
 	)
 	(segment
@@
 	)
 	(segment
-		(start 164.93025 46.08025)
-		(end 159.33125 40.48125)
-		(width 0.2)
-		(layer "F.Cu")
-		(net 2)
-	)
-	(segment
 		(start 154.66 57.15)
 		(end 153.34625 55.83625)
@@
 	)
 	(segment
-		(start 164.93025 47.77275)
-		(end 164.93025 46.08025)
-		(width 0.2)
-		(layer "F.Cu")
-		(net 2)
-	)
-	(segment
 		(start 131.1275 71.12)
 		(end 150.1775 71.12)
@@
 	)
 	(segment
+		(start 167.79 42.13)
+		(end 160.98 42.13)
+		(width 0.2)
+		(layer "B.Cu")
+		(net 2)
+	)
+	(segment
+		(start 169.2275 52.07)
+		(end 169.2275 43.5675)
+		(width 0.2)
+		(layer "B.Cu")
+		(net 2)
+	)
+	(segment
+		(start 169.2275 43.5675)
+		(end 167.79 42.13)
+		(width 0.2)
+		(layer "B.Cu")
+		(net 2)
+	)
+	(segment
+		(start 160.98 42.13)
+		(end 159.33125 40.48125)
+		(width 0.2)
+		(layer "B.Cu")
+		(net 2)
+	)
+	(segment
 		(start 153.34625 60.91625)
 		(end 141.085 60.91625)
@@
 	)
 	(segment
-		(start 128.55156 49.0055)
-		(end 126.020624 49.0055)
+		(start 143.00231 63.40066)
+		(end 136.655825 57.054175)
 		(width 0.2)
 		(layer "F.Cu")
@@
 	(segment
 		(start 143.00231 63.45625)
-		(end 128.55156 49.0055)
-		(width 0.2)
-		(layer "F.Cu")
-		(net 4)
-	)
-	(segment
-		(start 126.020624 49.0055)
-		(end 125.75925 48.744126)
-		(width 0.2)
-		(layer "F.Cu")
-		(net 4)
-	)
-	(segment
-		(start 125.75925 48.744126)
-		(end 125.75925 46.67687)
+		(end 143.00231 63.40066)
+		(width 0.2)
+		(layer "F.Cu")
+		(net 4)
+	)
+	(segment
+		(start 136.09654 56.49489)
+		(end 135.81511 56.49489)
+		(width 0.2)
+		(layer "F.Cu")
+		(net 4)
+	)
+	(segment
+		(start 136.655825 57.054175)
+		(end 136.09654 56.49489)
 		(width 0.2)
 		(layer "F.Cu")
@@
 		(net 4)
 	)
-	(segment
-		(start 125.75925 46.67687)
-		(end 127.03362 45.4025)
-		(width 0.2)
-		(layer "F.Cu")
+	(via
+		(at 135.81511 56.49489)
+		(size 0.6)
+		(drill 0.3)
+		(layers "F.Cu" "B.Cu")
+		(net 4)
+	)
+	(segment
+		(start 135.81511 56.49489)
+		(end 129.95 50.62978)
+		(width 0.2)
+		(layer "B.Cu")
+		(net 4)
+	)
+	(segment
+		(start 129.95 50.62978)
+		(end 129.95 47.24125)
+		(width 0.2)
+		(layer "B.Cu")
+		(net 4)
+	)
+	(segment
+		(start 129.95 47.24125)
+		(end 128.11125 45.4025)
+		(width 0.2)
+		(layer "B.Cu")
 		(net 4)
 	)
@@
 	)
 	(segment
-		(start 145.25625 72.23125)
-		(end 145.25625 49.8475)
-		(width 0.2)
-		(layer "B.Cu")
+		(start 140.55 54.2)
+		(end 140.55 50.74375)
+		(width 0.2)
+		(layer "F.Cu")
+		(net 8)
+	)
+	(segment
+		(start 140.55 50.74375)
+		(end 143.35125 47.9425)
+		(width 0.2)
+		(layer "F.Cu")
+		(net 8)
+	)
+	(segment
+		(start 142.818015 56.468015)
+		(end 140.55 54.2)
+		(width 0.2)
+		(layer "F.Cu")
+		(net 8)
+	)
+	(via
+		(at 142.818015 56.468015)
+		(size 0.6)
+		(drill 0.3)
+		(layers "F.Cu" "B.Cu")
 		(net 8)
 	)
 	(segment
 		(start 143.8275 73.66)
-		(end 145.25625 72.23125)
-		(width 0.2)
-		(layer "B.Cu")
-		(net 8)
-	)
-	(segment
-		(start 145.25625 49.8475)
-		(end 143.35125 47.9425)
-		(width 0.2)
-		(layer "B.Cu")
+		(end 143.8275 57.4775)
+		(width 0.2)
+		(layer "B.Cu")
+		(net 8)
+	)
+	(segment
+		(start 143.8275 57.4775)
+		(end 142.818015 56.468015)
+		(width 0.2)
+		(layer "B.Cu")
